File: schematics/Master Wiring Schematic/Master Wiring Schematic.kicad_sch (KiCad schematic)
At the start: 11 parts, among them J1 M5_Ring_Terminals, J2 Raspberry_Pi_4, J3 USB_A, J4 USB_B

Commit message: v1 of schematic complete
Parts:
- added SW1: Master_Switch_Pi_4, symbol Switch:SW_DPST_x2
Connections:
- net +5V: now also SW1.2 (B); no longer PS2.6 (+Vout)
- new net: PS2.6 (+Vout), SW1.1 (A)
Other:
- note added: "The Pi Camera circuitry is not shown; it connects to the Raspberry Pi 4 using a ribbon cable"
- moved on the sheet: F3, PS2

Commit message: Aesthetification of V1
Other:
- moved on the sheet: A1
Changed lines of the file:
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@@
 	(symbol
 		(lib_id "arduino-library:Arduino_Mega2560_R3_Shield")
-		(at 121.92 80.01 0)
+		(at 132.08 93.98 0)
 		(unit 1)
 		(body_style 1)
@@
 		(fields_autoplaced yes)
 		(property "Reference" "A1"
-			(at 121.92 140.97 0)
+			(at 132.08 154.94 0)
 			(show_name no)
 			(do_not_autoplace no)
@@
 		)
 		(property "Value" "Arduino_Mega2560_R3_Shield"
-			(at 121.92 143.51 0)
+			(at 132.08 157.48 0)
 			(show_name no)
 			(do_not_autoplace no)
@@
 		)
 		(property "Footprint" "PCM_arduino-library:Arduino_Mega2560_R3_Shield"
-			(at 121.92 153.67 0)
+			(at 132.08 167.64 0)
 			(hide yes)
 			(show_name no)
@@
 		)
 		(property "Datasheet" "https://docs.arduino.cc/hardware/mega-2560"
-			(at 121.92 149.86 0)
+			(at 132.08 163.83 0)
 			(hide yes)
 			(show_name no)
@@
 		)
 		(property "Description" "Shield for Arduino Mega 2560 R3"
-			(at 121.92 80.01 0)
+			(at 132.08 93.98 0)
 			(hide yes)
 			(show_name no)
